File: hardware/pragotron-master-clock-1.0.brd (EAGLE design)
At the start: 160 x 100 mm, 64 parts, among them IC1 ATSAMD21E18A-MU, IC2 AP2112K-3.3, IC3 MIC2288YD5-TR, IC4 DS3231MZ+, J1 USB-C, J2 TRMBLK_3.5MM_2P, J3 2X5_PITCH_1.27MMTH_NOKEY_UNSH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, Q1 N-MOSFET, Q2 N-MOSFET, Q3 N-MOSFET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

Commit message: board layout
Parts:
- S1: value TSA063G60-250 -> SKRPACE010; device BASTL_SWITCHES:TACTILE-SMT-SMALL-PADS -> BASTL_SWITCHES:SKRPACE010
- moved H3 114.4 mm to (45.7, 27.9)
- moved R5 110.0 mm to (42.4, 6.60), turned to 90 degrees
- moved H4 108.1 mm to (45.7, 2.54)
- moved R6 107.7 mm to (42.7, 23.9), turned to 270 degrees
- moved D4 106.2 mm to (44.7, 22.6), turned to 270 degrees
- moved D3 105.5 mm to (46.7, 8.38), turned to 270 degrees
- moved J3 102.6 mm to (39.4, 28.6), turned to 180 degrees
- moved D2 97.4 mm to (44.5, 8.38), turned to 270 degrees
- moved Q5 94.9 mm to (35.1, 13.0)
- moved LD3 93.5 mm to (30.2, 23.9), turned to 180 degrees
- moved R15 92.3 mm to (38.4, 20.3)
- moved Q4 89.7 mm to (38.4, 17.5), turned to 180 degrees
- moved S1 89.7 mm to (38.0, 24.6)
- moved R17 89.2 mm to (26.4, 18.5), turned to 90 degrees
- moved R12 87.2 mm to (38.4, 10.2), turned to 180 degrees
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Connections:
- net !RESET: now also S1.3, S1.4; no longer S1.1, S1.2
- net 32KHZ: now also IC1.8; no longer IC1.7
- net A: now also IC1.1; no longer IC1.17
- net B: now also IC1.2; no longer IC1.18
- net BOOST_EN: now also IC1.12
- net C: now also IC1.3; no longer IC1.19
- net D: now also IC1.4; no longer IC1.20
- net FAST/LEFT: now also IC1.17; no longer IC1.1
- net GND: now also S1.1, S1.2; no longer S1.3, S1.4
- net INT/SQW: now also IC1.7; no longer IC1.8
- net MINUTE/OK: now also IC1.19; no longer IC1.3
- net XFAST/RIGHT: now also IC1.18; no longer IC1.2
Other:
- board size 160 x 100 mm -> 48.3 x 30.5 mm
- board text added: "FAST"
- board text added: "GND VCC SCL SDA RX TX"
- board text added: "MIN. RESET"
- board text added: "OK"
- board text added: "PWR"
- board text added: "RST"
- board text added: "XFAST"

Commit message: finish board, add gerber, bom and cpl
Parts:
- moved R1 16.3 mm to (4.57, 6.99), turned to 180 degrees
- moved C14 7.64 mm to (19.1, 19.6)
- moved R14 3.66 mm to (29.5, 20.9)
- moved C13 1.56 mm to (27.8, 12.4), turned to 270 degrees
- moved R2 1.37 mm to (4.57, 8.64), turned to 180 degrees
- moved C11 1.37 mm to (27.8, 9.65)
- moved C8 1.10 mm to (5.41, 23.1)
- moved C7 0.97 mm to (7.16, 24.1)
- moved R16 0.76 mm to (19.1, 16.8)
- moved D2 0.76 mm to (44.5, 7.62), turned to 90 degrees
- moved D3 0.76 mm to (46.7, 7.62), turned to 90 degrees
- moved JP1 0.61 mm to (26.8, 23.9)
- moved F1 0.51 mm to (9.91, 18.5)
- moved J3 0.33 mm to (39.4, 28.2)
- moved C3 0.25 mm to (13.7, 12.2)
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Connections:
- removed net +3.3V: C12.1, C13.1, C14.1, C3.1, C4.1, IC1.30, IC1.9, IC2.5, IC4.2, J4.2, R16.2, R17.2
- net VDD: now also C12.1, C13.1, C14.1, C3.1, C4.1, IC1.30, IC1.9, IC2.5, IC4.2, J4.2, R16.2, R17.2
Routing:
- net 24V: track 0.00 -> 120.3 mm, vias 0 -> 5
- net VDD: track 0.00 -> 78.0 mm, vias 0 -> 4
- net RX: track 0.00 -> 65.1 mm, vias 0 -> 1
- net TX: track 0.00 -> 63.7 mm, vias 0 -> 1
- net GND: track 0.00 -> 52.5 mm, vias 0 -> 67
- net N$10: track 0.00 -> 46.9 mm, vias 0 -> 2
- net !RESET: track 0.00 -> 41.1 mm, vias 0 -> 2
- net D+: track 0.00 -> 41.1 mm, vias 0 -> 3
- net D-: track 0.00 -> 35.7 mm, vias 0 -> 3
- net OUT_2: track 0.00 -> 35.6 mm, vias 0 -> 2
- net SWCLK: track 0.00 -> 31.0 mm, vias 0 -> 2
- net OUT_1: track 0.00 -> 28.9 mm, vias 0 -> 1
- net SWDIO: track 0.00 -> 28.1 mm, vias 0 -> 1
- net MINUTE/OK: track 0.00 -> 26.1 mm, vias 0 -> 3
- net D: track 0.00 -> 23.4 mm, vias 0 -> 2
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- added copper zone on layer 1, net GND
- added copper zone on layer 16, net GND
Other:
- board text added: "*For future use/hacking:"
- board text added: "- for IPJ 0612 and others - 24V pulse source, using precise RTC with temperature compensation - power with a regular USB power brick - click FAST/XFAST to toggle scrolling through the numbers - click MINUTE RESET to set the current minute to 0s - hack using provided I2C and Serial ports"
- board text added: "Made by Vaclav Mach, open source github.com/xx0x/pragotron-master-clock"
- board text added: "Pragotron Master Clock"
- board text added: "Serial number:"
