File: hardware/pragotron-master-clock-1.0.brd (EAGLE design)
At the start: 48.3 x 30.5 mm, 64 parts, among them IC1 ATSAMD21E18A-MU, IC2 AP2112K-3.3, IC3 MIC2288YD5-TR, IC4 DS3231MZ+, J1 USB-C, J2 TRMBLK_3.5MM_2P, J3 2X5_PITCH_1.27MMTH_NOKEY_UNSH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, Q1 N-MOSFET, Q2 N-MOSFET, Q3 N-MOSFET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

Commit message: replace 22u with 10u caps (there are no 50V caps in 22u)
Parts:
- C10, C2, C4, C6, C8, C9: value 22u -> 10u
Changed lines of the file:
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@@
 <attribute name="WEB" value="" x="-35.052" y="-43.942" size="1.778" layer="27" rot="R270" display="off"/>
 </element>
-<element name="C10" library="BASTL_CAPACITORS" library_urn="urn:adsk.eagle:library:32978038" package="CAPACITOR0805" package3d_urn="urn:adsk.eagle:package:32978071/3" value="22u" x="35.052" y="20.574" smashed="yes">
+<element name="C10" library="BASTL_CAPACITORS" library_urn="urn:adsk.eagle:library:32978038" package="CAPACITOR0805" package3d_urn="urn:adsk.eagle:package:32978071/3" value="10u" x="35.052" y="20.574" smashed="yes">
 <attribute name="MAN" value="" x="74.422" y="-27.686" size="1.778" layer="27" display="off"/>
 <attribute name="MPN" value="" x="74.422" y="-27.686" size="1.778" layer="27" display="off"/>
@@
 <attribute name="WEB" value="" x="72.39" y="53.848" size="1.778" layer="27" rot="R90" display="off"/>
 </element>
-<element name="C2" library="BASTL_CAPACITORS" library_urn="urn:adsk.eagle:library:32978038" package="CAPACITOR0805" package3d_urn="urn:adsk.eagle:package:32978071/3" value="22u" x="9.8298" y="15.24" smashed="yes" rot="R270">
+<element name="C2" library="BASTL_CAPACITORS" library_urn="urn:adsk.eagle:library:32978038" package="CAPACITOR0805" package3d_urn="urn:adsk.eagle:package:32978071/3" value="10u" x="9.8298" y="15.24" smashed="yes" rot="R270">
 <attribute name="MAN" value="" x="-38.4302" y="-5.08" size="1.778" layer="27" rot="R270" display="off"/>
 <attribute name="MPN" value="" x="-38.4302" y="-5.08" size="1.778" layer="27" rot="R270" display="off"/>
@@
 <attribute name="WEB" value="" x="-39.624" y="-3.048" size="1.778" layer="27" rot="R270" display="off"/>
 </element>
-<element name="C4" library="BASTL_CAPACITORS" library_urn="urn:adsk.eagle:library:32978038" package="CAPACITOR0805" package3d_urn="urn:adsk.eagle:package:32978071/3" value="22u" x="16.002" y="11.938" smashed="yes" rot="R270">
+<element name="C4" library="BASTL_CAPACITORS" library_urn="urn:adsk.eagle:library:32978038" package="CAPACITOR0805" package3d_urn="urn:adsk.eagle:package:32978071/3" value="10u" x="16.002" y="11.938" smashed="yes" rot="R270">
 <attribute name="MAN" value="" x="-32.258" y="-12.192" size="1.778" layer="27" rot="R270" display="off"/>
 <attribute name="MPN" value="" x="-32.258" y="-12.192" size="1.778" layer="27" rot="R270" display="off"/>
@@
 <attribute name="WEB" value="" x="33.274" y="-33.02" size="1.778" layer="27" display="off"/>
 </element>
-<element name="C6" library="BASTL_CAPACITORS" library_urn="urn:adsk.eagle:library:32978038" package="CAPACITOR0805" package3d_urn="urn:adsk.eagle:package:32978071/3" value="22u" x="14.224" y="18.542" smashed="yes">
+<element name="C6" library="BASTL_CAPACITORS" library_urn="urn:adsk.eagle:library:32978038" package="CAPACITOR0805" package3d_urn="urn:adsk.eagle:package:32978071/3" value="10u" x="14.224" y="18.542" smashed="yes">
 <attribute name="MAN" value="" x="42.164" y="-29.718" size="1.778" layer="27" display="off"/>
 <attribute name="MPN" value="" x="42.164" y="-29.718" size="1.778" layer="27" display="off"/>
@@
 <attribute name="WEB" value="" x="-46.1772" y="1.27" size="1.778" layer="27" rot="R270" display="off"/>
 </element>
-<element name="C8" library="BASTL_CAPACITORS" library_urn="urn:adsk.eagle:library:32978038" package="CAPACITOR0805" package3d_urn="urn:adsk.eagle:package:32978071/3" value="22u" x="5.4102" y="23.0886" smashed="yes" rot="R270">
+<element name="C8" library="BASTL_CAPACITORS" library_urn="urn:adsk.eagle:library:32978038" package="CAPACITOR0805" package3d_urn="urn:adsk.eagle:package:32978071/3" value="10u" x="5.4102" y="23.0886" smashed="yes" rot="R270">
 <attribute name="MAN" value="" x="-42.8498" y="-8.6614" size="1.778" layer="27" rot="R270" display="off"/>
 <attribute name="MPN" value="" x="-42.8498" y="-8.6614" size="1.778" layer="27" rot="R270" display="off"/>
@@
 <attribute name="WEB" value="" x="-42.8498" y="-8.6614" size="1.778" layer="27" rot="R270" display="off"/>
 </element>
-<element name="C9" library="BASTL_CAPACITORS" library_urn="urn:adsk.eagle:library:32978038" package="CAPACITOR0805" package3d_urn="urn:adsk.eagle:package:32978071/3" value="22u" x="35.052" y="9.906" smashed="yes" rot="R180">
+<element name="C9" library="BASTL_CAPACITORS" library_urn="urn:adsk.eagle:library:32978038" package="CAPACITOR0805" package3d_urn="urn:adsk.eagle:package:32978071/3" value="10u" x="35.052" y="9.906" smashed="yes" rot="R180">
 <attribute name="MAN" value="" x="-0.508" y="58.166" size="1.778" layer="27" rot="R180" display="off"/>
 <attribute name="MPN" value="" x="-0.508" y="58.166" size="1.778" layer="27" rot="R180" display="off"/>

Commit message: small fixes
Parts:
- added HW1: SPC_M3X5X8_IA_M, BASTL_MECHANICAL:SPC_M3X5X8_IA_M
- moved D2 1.05 mm to (44.7, 8.64)
- moved D3 1.02 mm to (46.7, 8.64)
- moved D4 0.79 mm to (44.7, 21.8)
- moved D5 0.76 mm to (46.7, 21.8)
Routing:
- net 24V: track 120.3 -> 122.5 mm
- net OUT_1: track 28.9 -> 27.0 mm
- net GND: track 52.5 -> 53.3 mm
Other:
- board text added: "- for IPJ 0612 and others - 24V pulse source, using precise RTC with a temperature compensation - power with a regular USB power brick - click FAST/XFAST to toggle scrolling through the numbers - click MINUTE RESET to set the current minute to 0s - hack using provided I2C and Serial ports"
- board text removed: "- for IPJ 0612 and others - 24V pulse source, using precise RTC with temperature compensation - power with a regular USB power brick - click FAST/XFAST to toggle scrolling through the numbers - click MINUTE RESET to set the current minute to 0s - hack using provided I2C and Serial ports"

Commit message: small fixes
Parts:
- removed HW1: SPC_M3X5X8_IA_M, BASTL_MECHANICAL:SPC_M3X5X8_IA_M
Other:
- board text added: "Note:"
- board text removed: "Serial number:"
Changed lines of the file:
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@@
 <grid distance="20" unitdist="mil" unit="mil" style="lines" multiple="1" display="yes" altdistance="1" altunitdist="mil" altunit="mil"/>
 <layers>
-<layer number="1" name="Top" color="4" fill="1" visible="no" active="yes"/>
+<layer number="1" name="Top" color="4" fill="1" visible="yes" active="yes"/>
 <layer number="2" name="Route2" color="16" fill="1" visible="no" active="no"/>
 <layer number="3" name="Route3" color="17" fill="1" visible="no" active="no"/>
@@
 <layer number="14" name="Route14" color="22" fill="1" visible="no" active="no"/>
 <layer number="15" name="Route15" color="23" fill="1" visible="no" active="no"/>
-<layer number="16" name="Bottom" color="1" fill="1" visible="no" active="yes"/>
+<layer number="16" name="Bottom" color="1" fill="1" visible="yes" active="yes"/>
 <layer number="17" name="Pads" color="2" fill="1" visible="yes" active="yes"/>
 <layer number="18" name="Vias" color="2" fill="1" visible="yes" active="yes"/>
-<layer number="19" name="Unrouted" color="6" fill="1" visible="no" active="yes"/>
+<layer number="19" name="Unrouted" color="6" fill="1" visible="yes" active="yes"/>
 <layer number="20" name="Dimension" color="24" fill="1" visible="yes" active="yes"/>
-<layer number="21" name="tPlace" color="7" fill="1" visible="no" active="yes"/>
+<layer number="21" name="tPlace" color="7" fill="1" visible="yes" active="yes"/>
 <layer number="22" name="bPlace" color="7" fill="1" visible="yes" active="yes"/>
-<layer number="23" name="tOrigins" color="15" fill="1" visible="no" active="yes"/>
+<layer number="23" name="tOrigins" color="15" fill="1" visible="yes" active="yes"/>
 <layer number="24" name="bOrigins" color="15" fill="1" visible="yes" active="yes"/>
-<layer number="25" name="tNames" color="7" fill="1" visible="no" active="yes"/>
+<layer number="25" name="tNames" color="7" fill="1" visible="yes" active="yes"/>
 <layer number="26" name="bNames" color="7" fill="1" visible="yes" active="yes"/>
 <layer number="27" name="tValues" color="7" fill="1" visible="no" active="yes"/>
 <layer number="28" name="bValues" color="7" fill="1" visible="no" active="yes"/>
 <layer number="29" name="tStop" color="7" fill="3" visible="no" active="yes"/>
-<layer number="30" name="bStop" color="7" fill="6" visible="yes" active="yes"/>
+<layer number="30" name="bStop" color="7" fill="6" visible="no" active="yes"/>
 <layer number="31" name="tCream" color="7" fill="4" visible="no" active="yes"/>
 <layer number="32" name="bCream" color="7" fill="5" visible="no" active="yes"/>
@@
 <layer number="37" name="tTest" color="7" fill="1" visible="no" active="yes"/>
 <layer number="38" name="bTest" color="7" fill="1" visible="no" active="yes"/>
-<layer number="39" name="tKeepout" color="4" fill="11" visible="no" active="yes"/>
-<layer number="40" name="bKeepout" color="1" fill="11" visible="no" active="yes"/>
-<layer number="41" name="tRestrict" color="4" fill="10" visible="no" active="yes"/>
-<layer number="42" name="bRestrict" color="1" fill="10" visible="no" active="yes"/>
+<layer number="39" name="tKeepout" color="4" fill="11" visible="yes" active="yes"/>
+<layer number="40" name="bKeepout" color="1" fill="11" visible="yes" active="yes"/>
+<layer number="41" name="tRestrict" color="4" fill="10" visible="yes" active="yes"/>
+<layer number="42" name="bRestrict" color="1" fill="10" visible="yes" active="yes"/>
 <layer number="43" name="vRestrict" color="2" fill="10" visible="no" active="yes"/>
 <layer number="44" name="Drills" color="7" fill="1" visible="no" active="yes"/>
@@
 <layer number="49" name="Reference" color="7" fill="1" visible="no" active="yes"/>
 <layer number="50" name="dxf" color="7" fill="1" visible="no" active="no"/>
-<layer number="51" name="tDocu" color="7" fill="1" visible="no" active="yes"/>
+<layer number="51" name="tDocu" color="7" fill="1" visible="yes" active="yes"/>
 <layer number="52" name="bDocu" color="7" fill="1" visible="yes" active="yes"/>
 <layer number="53" name="tGND_GNDA" color="7" fill="1" visible="no" active="no"/>
@@
 <text x="42.672" y="1.016" size="0.8128" layer="22" ratio="15" rot="MR0">Made by Vaclav Mach, open source
 github.com/xx0x/pragotron-master-clock</text>
-<circle x="12.6746" y="21.59" radius="0.851940625" width="0.1524" layer="22"/>
-<text x="12.6746" y="21.59" size="0.7112" layer="22" ratio="15" rot="MR0" align="center">OK</text>
-<circle x="15.0876" y="21.59" radius="0.851940625" width="0.1524" layer="22"/>
-<wire x1="15.5956" y1="21.59" x2="14.5796" y2="21.59" width="0.1524" layer="22"/>
-<wire x1="14.9606" y1="21.971" x2="14.5796" y2="21.59" width="0.1524" layer="22"/>
-<wire x1="14.5796" y1="21.59" x2="14.9606" y2="21.209" width="0.1524" layer="22"/>
-<circle x="17.3736" y="21.59" radius="0.851940625" width="0.1524" layer="22"/>
-<wire x1="16.8656" y1="21.59" x2="17.8816" y2="21.59" width="0.1524" layer="22"/>
-<wire x1="17.5006" y1="21.209" x2="17.8816" y2="21.59" width="0.1524" layer="22"/>
-<wire x1="17.8816" y1="21.59" x2="17.5006" y2="21.971" width="0.1524" layer="22"/>
-<text x="18.2118" y="23.114" size="0.8128" layer="22" ratio="15" rot="MR0">For future use/hacking:</text>
+<circle x="12.6746" y="21.082" radius="0.851940625" width="0.1524" layer="22"/>
+<text x="12.6746" y="21.082" size="0.7112" layer="22" ratio="15" rot="MR0" align="center">OK</text>
+<circle x="15.0876" y="21.082" radius="0.851940625" width="0.1524" layer="22"/>
+<wire x1="15.5956" y1="21.082" x2="14.5796" y2="21.082" width="0.1524" layer="22"/>
+<wire x1="14.9606" y1="21.463" x2="14.5796" y2="21.082" width="0.1524" layer="22"/>
+<wire x1="14.5796" y1="21.082" x2="14.9606" y2="20.701" width="0.1524" layer="22"/>
+<circle x="17.3736" y="21.082" radius="0.851940625" width="0.1524" layer="22"/>
+<wire x1="16.8656" y1="21.082" x2="17.8816" y2="21.082" width="0.1524" layer="22"/>
+<wire x1="17.5006" y1="20.701" x2="17.8816" y2="21.082" width="0.1524" layer="22"/>
+<wire x1="17.8816" y1="21.082" x2="17.5006" y2="21.463" width="0.1524" layer="22"/>
+<text x="18.2118" y="22.606" size="0.8128" layer="22" ratio="15" rot="MR0">For future use/hacking:</text>
 <rectangle x1="25.654" y1="20.066" x2="42.672" y2="23.876" layer="22"/>
-<text x="42.672" y="24.384" size="0.8128" layer="22" ratio="15" rot="MR0">Serial number:</text>
+<text x="42.672" y="24.384" size="0.8128" layer="22" ratio="15" rot="MR0">Note:</text>
 <text x="18.2118" y="24.384" size="0.8128" layer="22" ratio="15" rot="MR0">Version: 1.0</text>
 </plain>
@@
 <attribute name="MAN" value="DIOTEC SEMICONDUCTOR " x="2.7686" y="-37.8714" size="1.778" layer="27" rot="R270" display="off"/>
 <attribute name="MPN" value="SL1M" x="2.7686" y="-37.8714" size="1.778" layer="27" rot="R270" display="off"/>
-<attribute name="NAME" x="44.7294" y="24.638" size="0.8" layer="25" font="fixed" ratio="15" align="center"/>
+<attribute name="NAME" x="44.6532" y="25.0698" size="0.8" layer="25" font="fixed" ratio="15" align="center"/>
 <attribute name="ODOO" value="D_SL1M_SOD123" x="2.7686" y="-37.8714" size="1.778" layer="27" rot="R270" display="off"/>
 <attribute name="PRICE" value="0.5" x="2.7686" y="-37.8714" size="1.778" layer="27" rot="R270" display="off"/>
@@
 <attribute name="MAN" value="DIOTEC SEMICONDUCTOR " x="-1.524" y="6.604" size="1.778" layer="27" rot="R270" display="off"/>
 <attribute name="MPN" value="SL1M" x="-1.524" y="6.604" size="1.778" layer="27" rot="R270" display="off"/>
-<attribute name="NAME" x="46.736" y="24.4348" size="0.8" layer="25" font="fixed" ratio="15" align="center"/>
+<attribute name="NAME" x="46.7106" y="25.0444" size="0.8" layer="25" font="fixed" ratio="15" align="center"/>
 <attribute name="ODOO" value="D_SL1M_SOD123" x="-1.524" y="6.604" size="1.778" layer="27" rot="R270" display="off"/>
 <attribute name="PRICE" value="0.5" x="-1.524" y="6.604" size="1.778" layer="27" rot="R270" display="off"/>
@@
 <attribute name="VALUE" x="35.52725" y="21.687940625" size="0.8128" layer="27" ratio="15"/>
 </element>
-<element name="HW1" library="BASTL_MECHANICAL" library_urn="urn:adsk.eagle:library:32977656" package="SPC_M3X5X8_IA_M" package3d_urn="urn:adsk.eagle:package:42477236/2" value="SPC_M3X5X8_IA_M" x="45.72" y="2.54" smashed="yes"/>
 </elements>
 <signals>
